File: PCB/OpenSpritzer/OpenSpritzer.kicad_pcb (KiCad board)
At the start: 2 copper layers, 16 parts, among them J1 foot_pedal, J2 24V_in, J3 to_solenoid, Q1 Q_NPN_Darlington_EBC, SW1 SW_DPDT_x2

Commit message: update board. Main is done
Parts:
- added ?: , Mounting_Holes:MountingHole_3.2mm_M3, F.Cu at (107.0, 125.5)
- added ?: , Mounting_Holes:MountingHole_3.2mm_M3, F.Cu at (107.0, 87.0)
- Q1: value Q_NPN_Darlington_EBC -> NPN_Darlington_EBC
Routing:
- net Net-(A1-Pad19): track 73.3 -> 77.7 mm
- net Net-(A1-Pad27): track 110.0 -> 110.6 mm
Other:
- board outline added: 48 x 49 mm
- board text added: "+"
- board text added: "-"

Commit message: board with hardware licence and links
Other:
- board text added: "OpenSpritzer v0.01 20180727 By AM Chagas Released under CERN OHL v1.2"
- board text added: "Source: https://open-labware.net/ projects/openspritzer/"
Changed lines of the file:
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@@
   (general
     (thickness 1.6)
-    (drawings 11)
+    (drawings 13)
     (tracks 99)
     (zones 0)
@@
   (layers
     (0 F.Cu signal hide)
-    (31 B.Cu signal)
+    (31 B.Cu signal hide)
     (32 B.Adhes user)
     (33 F.Adhes user)
@@
     (pad 1 np_thru_hole circle (at 0 0) (size 3.2 3.2) (drill 3.2) (layers *.Cu *.Mask))
   )
+  (gr_text "Source:\nhttps://open-labware.net/\nprojects/openspritzer/" (at 107.5 122.5 90) (layer B.SilkS)
+    (effects (font (size 1.5 1.5) (thickness 0.3)) (justify left))
+  )
+  (gr_text "OpenSpritzer v0.01\n20180727\nBy AM Chagas\nReleased under CERN OHL v1.2" (at 120.5 106.5 90) (layer B.SilkS)
+    (effects (font (size 1.5 1.5) (thickness 0.3)))
+  )
   (gr_line (start 83 130) (end 83.5 130) (layer Edge.Cuts) (width 0.2))
