File: PCB/OpenSpritzer v1.02/OpenSpritzer_1.02.kicad_pcb (KiCad board)
At the start: 2 copper layers, 62.5 x 75 mm, 30 parts

Commit message: v1.02
Parts:
- removed the ? at (124.8, 110.0)
- added G***: LOGO, Maxime:logo 400, F.Cu at (135.1, 69.2)
- ?: footprint Potentiometers:Potentiometer_Alps_RK09K_Horizontal -> Maxime:Potentiometer
- moved ? 7.74 mm to (144.4, 143.5)
Connections:
- ? pad 1: GNDREF -> Net-(C1-Pad1)
- ? pad 2: Net-(C1-Pad1) -> GNDREF
Routing:
- net Net-(Q1-Pad1): track 52.5 -> 61.4 mm
- net Net-(R1-Pad1): track 19.0 -> 26.3 mm
- net Net-(A1-Pad27): track 115.9 -> 120.5 mm, vias 0 -> 1
- net Net-(C1-Pad1): track 114.6 -> 115.7 mm

Commit message: V 1.02
Parts:
- removed G***: LOGO, Maxime:logo 400
Routing:
- net GNDREF: track 0.00 -> 112.8 mm
- net Net-(Q1-Pad1): vias 0 -> 1

Commit message: V 1.02
Parts:
- ?: value 1 kΩ -> 1kΩ Potentiometer
- moved ? 12.7 mm to (147.5, 134.6), turned to 180 degrees
Connections:
- ? pad 1: Net-(Q1-Pad1) -> GNDREF
Routing:
- net GNDREF: track 112.8 -> 96.5 mm
- net Net-(D1-Pad2): track 4.53 -> 18.0 mm
- net Net-(R2-Pad2): track 37.2 -> 27.8 mm, vias 0 -> 1
- net Net-(Q1-Pad1): vias 1 -> 0
Other:
- board text added: "Source: https://open-labware.net/projects/openspritzer"
- board text removed: "Source: https://open-labware.net/projects/openspritzer/"
