File: PCB/OpenSpritzer v1.02/_autosave-OpenSpritzer_1.02.kicad_pcb (KiCad board)
At the start: 2 copper layers, 62.5 x 75 mm, 29 parts

Commit message: v 1.02
Parts:
- moved ? 1.76 mm to (135.3, 96.9)
Changed lines of the file:
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@@
       (effects (font (size 1 1) (thickness 0.15)))
     )
-    (fp_text value "24V in" (at 17.975 0.125 180) (layer F.SilkS)
-      (effects (font (size 1.25 1.25) (thickness 0.15)))
+    (fp_text value "24V in" (at 17.95 -1.125 180) (layer F.SilkS)
+      (effects (font (size 1.3 1.3) (thickness 0.2)))
     )
     (fp_line (start 14.02 -4.5) (end 0.32 -4.5) (layer F.Fab) (width 0.1))
@@
     )
     (fp_text value "Arduino Nano v3.0" (at 7.65 17.675) (layer F.SilkS)
-      (effects (font (size 1.25 1.25) (thickness 0.15)))
+      (effects (font (size 1.3 1.3) (thickness 0.2)))
     )
     (fp_text user "" (at 3 18) (layer F.Fab)
@@
   )
   (module "Maxime:new_logo 2500" (layer F.Cu)
-    (at 135.5 95.15)
+    (at 135.275 96.9)
     (fp_text reference "" (at 0 0) (layer F.SilkS) hide
       (effects (font (size 1.524 1.524) (thickness 0.3)))
@@
     (effects (font (size 1.5 1.5) (thickness 0.125)) (justify left))
   )
-  (gr_text "by AM Chagas & MJY Zimmermann\nReleased under CERN OHL v1.2" (at 115.225 85.225) (layer F.SilkS)
+  (gr_text "by AM Chagas & MJY Zimmermann\nReleased under CERN OHL v1.2" (at 115.175 85.55) (layer F.SilkS)
     (effects (font (size 1.25 1.25) (thickness 0.125)) (justify left))
   )
-  (gr_text "Source:\nhttps://open-labware.net/projects/openspritzer" (at 115.1 88.85) (layer F.SilkS)
+  (gr_text "Source:\nhttps://open-labware.net/projects/openspritzer" (at 115.125 89.85) (layer F.SilkS)
     (effects (font (size 1 1) (thickness 0.125)) (justify left))
   )
