File: Printed Circuit Board/OpenSpritzer v1.2/_autosave-OpenSpritzer_1.2.kicad_pcb (KiCad board)
At the start: 2 copper layers, 62.5 x 75 mm, 29 parts

Commit message: V1.2
Parts:
- removed the ? at (100.0, 150.0)
- moved ? 1.76 mm to (135.3, 96.9)
Other:
- board text added: "2018.10.10"
- board text added: "OpenSpritzer v1.2"
- board text removed: "2018.09.10"
- board text removed: "OpenSpritzer v1.02"
Changed lines of the file:
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@@
     (tracks 202)
     (zones 0)
-    (modules 29)
+    (modules 28)
     (nets 43)
   )
@@
       (effects (font (size 1 1) (thickness 0.15)))
     )
-    (fp_text value "24V in" (at 17.975 0.125 180) (layer F.SilkS)
-      (effects (font (size 1.25 1.25) (thickness 0.15)))
+    (fp_text value "24V in" (at 17.95 -1.125 180) (layer F.SilkS)
+      (effects (font (size 1.3 1.3) (thickness 0.2)))
     )
     (fp_line (start 14.02 -4.5) (end 0.32 -4.5) (layer F.Fab) (width 0.1))
@@
   )
   (module MountingHole:MountingHole_6.4mm_M6 (layer F.Cu)
-    (at 100 150)
-    (descr "Mounting Hole 6.4mm, no annular, M6")
-    (tags "mounting hole 6.4mm no annular m6")
-    (attr virtual)
-    (fp_text reference "" (at 0 -7.4) (layer F.SilkS)
-      (effects (font (size 1 1) (thickness 0.15)))
-    )
-    (fp_text value "" (at 0 7.4) (layer F.Fab)
-      (effects (font (size 1 1) (thickness 0.15)))
-    )
-    (fp_circle (center 0 0) (end 6.65 0) (layer F.CrtYd) (width 0.05))
-    (fp_circle (center 0 0) (end 6.4 0) (layer Cmts.User) (width 0.15))
-    (fp_text user %R (at 0.3 0) (layer F.Fab)
-      (effects (font (size 1 1) (thickness 0.15)))
-    )
-    (pad 1 np_thru_hole circle (at 0 0) (size 6.4 6.4) (drill 6.4) (layers *.Cu *.Mask))
-  )
-  (module MountingHole:MountingHole_6.4mm_M6 (layer F.Cu)
     (at 100 75)
     (descr "Mounting Hole 6.4mm, no annular, M6")
@@
       (rotate (xyz 0 0 0))
     )
+    (model ${KISYS3DMOD}/conn_rf/bnc_90_1-1337543-0.wrl
+      (offset (xyz 0 7.5 0))
+      (scale (xyz 1 1 1))
+      (rotate (xyz 0 0 180))
+    )
   )
   (module Modules:Arduino_Nano_WithMountingHoles (layer F.Cu)
@@
     )
     (fp_text value "Arduino Nano v3.0" (at 7.65 17.675) (layer F.SilkS)
-      (effects (font (size 1.25 1.25) (thickness 0.15)))
+      (effects (font (size 1.3 1.3) (thickness 0.2)))
     )
     (fp_text user "" (at 3 18) (layer F.Fab)
@@
     (pad "" np_thru_hole circle (at 0 38.1 270) (size 1.78 1.78) (drill 1.78) (layers *.Cu *.Mask))
     (model ${KISYS3DMOD}/Library_3D_shield_arduino/Shield_Arduino/Arduino_Nano/nano3.wrl
-      (offset (xyz 16.5 -39.4 2.5))
+      (offset (xyz 16.5 -39.4 9.6))
       (scale (xyz 1 1 1))
       (rotate (xyz -90 0 -90))
     )
+    (model ${KISYS3DMOD}/Connector_PinSocket_2.54mm.3dshapes/PinSocket_1x15_P2.54mm_Vertical.wrl
+      (at (xyz 0 0 0))
+      (scale (xyz 1 1 1))
+      (rotate (xyz 0 0 0))
+    )
+    (model ${KISYS3DMOD}/Connector_PinSocket_2.54mm.3dshapes/PinSocket_1x15_P2.54mm_Vertical.wrl
+      (offset (xyz 15.25 0 0))
+      (scale (xyz 1 1 1))
+      (rotate (xyz 0 0 0))
+    )
   )
   (module Diodes_THT:D_DO-35_SOD27_P7.62mm_Horizontal (layer F.Cu)
@@
       (rotate (xyz 0 0 0))
     )
+    (model ${KISYS3DMOD}/conn_rf/bnc_90_1-1337543-0.wrl
+      (offset (xyz 0 7.5 0))
+      (scale (xyz 1 1 1))
+      (rotate (xyz 0 0 180))
+    )
   )
   (module "Maxime:new_logo 2500" (layer F.Cu)
-    (at 135.5 95.15)
+    (at 135.275 96.9)
     (fp_text reference "" (at 0 0) (layer F.SilkS) hide
       (effects (font (size 1.524 1.524) (thickness 0.3)))
@@
   (gr_line (start 144.4 119.25) (end 146.6 119.25) (layer F.SilkS) (width 0.2))
   (gr_line (start 144.4 112.15) (end 144.4 119.25) (layer F.SilkS) (width 0.2))
-  (gr_text 2018.09.10 (at 137.4 81.55) (layer F.SilkS)
+  (gr_text 2018.10.10 (at 136 81.475) (layer F.SilkS)
     (effects (font (size 1.5 1.5) (thickness 0.125)) (justify left))
   )
-  (gr_text "by AM Chagas & MJY Zimmermann\nReleased under CERN OHL v1.2" (at 115.225 85.225) (layer F.SilkS)
+  (gr_text "by AM Chagas & MJY Zimmermann\nReleased under CERN OHL v1.2" (at 115.175 85.55) (layer F.SilkS)
     (effects (font (size 1.25 1.25) (thickness 0.125)) (justify left))
   )
-  (gr_text "Source:\nhttps://open-labware.net/projects/openspritzer" (at 115.1 88.85) (layer F.SilkS)
+  (gr_text "Source:\nhttps://open-labware.net/projects/openspritzer" (at 115.125 90.325) (layer F.SilkS)
     (effects (font (size 1 1) (thickness 0.125)) (justify left))
   )
-  (gr_text "OpenSpritzer v1.02\n\n" (at 126.8 80.95) (layer F.SilkS)
+  (gr_text "OpenSpritzer v1.2\n\n" (at 127.3 80.925) (layer F.SilkS)
     (effects (font (size 3 3) (thickness 0.5)))
   )
