File: Printed Circuit Board/OpenSpritzer v1.3/OpenSpritzer_1.3.kicad_pcb (KiCad board)
At the start: 2 copper layers, 57.5 x 85 mm, 30 parts

Commit message: v1.3
Parts:
- ?: footprint Maxime:maxi_PINHEAD1-2 -> Maxime:JST_XH_B03B-XH-A_03x2.50mm_Straight
- ? (x2): footprint Maxime:maxi_PINHEAD1-2 -> Maxime:JST_XH_B02B-XH-A_02x2.50mm_Straight
- moved ? 2.02 mm to (133.0, 85.5)
- moved ? 1.03 mm to (154.5, 81.7)
- moved ? 0.56 mm to (154.5, 131.9)
- moved ? 0.56 mm to (154.5, 141.7)
Routing:
- net Net-(C1-Pad1): track 120.1 -> 126.4 mm
- net Net-(D1-Pad2): track 4.94 -> 6.91 mm
- net Net-(D3-Pad2): track 59.5 -> 58.3 mm
Other:
- board text added: "Source: https://github.com/BadenLab"
- board text added: "by MJY Zimmermann & AM Chagas Released under CERN OHL v1.2"
- board text removed: "Source: https://open-labware.net/projects/openspritzer"
- board text removed: "by AM Chagas & MJY Zimmermann Released under CERN OHL v1.2"
